File: snes_feram.sch (KiCad schematic (older format))
At the start: 33 parts, among them CON1 SNES-EDGE, J1 Conn_01x23_Male, J2 Conn_01x23_Male, SW1 SW_DIP_x04, U1 4081, U2 4071, U3 27C322, U5 74LS245, U6 74LS245, U7 74LS139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

Commit message: Forgot to add protection resistor to LED
Parts:
- added R5: 1K, Resistor_THT:R_Axial_DIN0207_L6.3mm_D2.5mm_P7.62mm_Horizontal, symbol Device:R
Connections:
- net GND: now also R5.2; no longer D1.1 (K)
- new net: D1.1 (K), R5.1
Changed lines of the file:
@@
 EESchema Schematic File Version 4
-LIBS:snes_multicart-cache
+LIBS:snes_feram-cache
 EELAYER 30 0
 EELAYER END
@@
 	2950 7050 2950 7600
 Wire Wire Line
-	2950 7600 1650 7600
-Wire Wire Line
 	1650 7600 1650 7650
 Connection ~ 1650 7650
@@
 Wire Notes Line
 	550  8100 10850 8100
+$Comp
+L Device:R R5
+U 1 1 5F973EE2
+P 2450 7600
+F 0 "R5" V 2243 7600 50  0000 C CNN
+F 1 "1K" V 2334 7600 50  0000 C CNN
+F 2 "Resistor_THT:R_Axial_DIN0207_L6.3mm_D2.5mm_P7.62mm_Horizontal" V 2380 7600 50  0001 C CNN
+F 3 "~" H 2450 7600 50  0001 C CNN
+	1    2450 7600
+	0    1    1    0
+$EndComp
+Wire Wire Line
+	2600 7600 2950 7600
+Wire Wire Line
+	2300 7600 1650 7600
 $EndSCHEMATC
